File: hardware/rgb-led-matrix-v2.sch (KiCad schematic (older format))
At the start: 152 parts, among them J1 AKL_5_2, P1 CONN_01X02, P2 CON-SENSOR, Q1 2N7002P, U1 XMC1100-16, U2 DRILL, U3 DRILL, U4 DRILL, U5 DRILL

Commit message: changed schematic ws2813b led
Parts:
- removed LED1, LED10, LED11, LED12, LED13, LED14, LED15, LED16, LED17, LED18, LED19, LED2, LED20, LED21, LED22, LED23, LED24, LED25, LED26, LED27, LED28, LED29, LED3, LED30, LED31, LED32, LED33, LED34, LED35, LED36, LED37, LED38, LED39, LED4, LED40, LED41, LED42, LED43, LED44, LED45, LED46, LED47, LED48, LED49, LED5, LED50, LED51, LED52, LED53, LED54, LED55, LED56, LED57, LED58, LED59, LED6, LED60, LED61, LED62, LED63, LED64, LED7, LED8, LED9: WS2812B_LED, kicad-libraries:WS2812B_LED, symbol tinkerforge:WS2812B_LED
- added U10, U11, U12, U13, U14, U15, U16, U17, U18, U19, U20, U21, U22, U23, U24, U25, U26, U27, U28, U29, U30, U31, U32, U33, U34, U35, U36, U37, U38, U39, U40, U41, U42, U43, U44, U45, U46, U47, U48, U49, U50, U51, U52, U53, U54, U55, U56, U57, U58, U59, U6, U60, U61, U62, U63, U64, U65, U66, U67, U68, U69, U7, U8, U9: WS2813B, kicad-libraries:WS2813B, symbol tinkerforge:WS2813B
Connections:
- net GND: now also C10.1, C11.1, C12.1, C13.1, C14.1, C15.1, C16.1, C17.1, C18.1, C19.1, C20.1, C21.1, C22.1, C23.1, C24.1, C25.1, C26.1, C27.1, C28.1, C29.1, C30.1, C31.1, C32.1, C33.1, C34.1, C35.1, C36.1, C37.1, C38.1, C39.1, C40.1, C41.1, C42.1, C43.1, C44.1, C45.1, C46.1, C47.1, C48.1, C49.1, C50.1, C51.1, C52.1, C53.1, C54.1, C55.1, C56.1, C57.1, C58.1, C59.1, C6.1, C60.1, C61.1, C62.1, C63.1, C64.1, C65.1, C66.1, C67.1, C68.1, C69.1, C7.1, C8.1, C9.1, U10.5 (GND), U11.5 (GND), U12.5 (GND), U13.5 (GND), U14.5 (GND), U15.5 (GND), U16.5 (GND), U17.5 (GND), U18.5 (GND), U19.5 (GND), U20.5 (GND), U21.5 (GND), U22.5 (GND), U23.5 (GND), U24.5 (GND), U25.5 (GND), U26.5 (GND), U27.5 (GND), U28.5 (GND), U29.5 (GND), U30.5 (GND), U31.5 (GND), U32.5 (GND), U33.5 (GND), U34.5 (GND), U35.5 (GND), U36.5 (GND), U37.5 (GND), U38.5 (GND), U39.5 (GND), U40.5 (GND), U41.5 (GND), U42.5 (GND), U43.5 (GND), U44.5 (GND), U45.5 (GND), U46.5 (GND), U47.5 (GND), U48.5 (GND), U49.5 (GND), U50.5 (GND), U51.5 (GND), U52.5 (GND), U53.5 (GND), U54.5 (GND), U55.5 (GND), U56.5 (GND), U57.5 (GND), U58.5 (GND), U59.5 (GND), U6.5 (GND), U6.6 (BIN), U60.5 (GND), U61.5 (GND), U62.5 (GND), U63.5 (GND), U64.5 (GND), U65.5 (GND), U66.5 (GND), U67.5 (GND), U68.5 (GND), U69.5 (GND), U7.5 (GND), U8.5 (GND), U9.5 (GND); no longer C10.2, C11.2, C12.2, C13.2, C14.2, C15.2, C16.2, C17.2, C18.2, C19.2, C20.2, C21.2, C22.2, C23.2, C24.2, C25.2, C26.2, C27.2, C28.2, C29.2, C30.2, C31.2, C32.2, C33.2, C34.2, C35.2, C36.2, C37.2, C38.2, C39.2, C40.2, C41.2, C42.2, C43.2, C44.2, C45.2, C46.2, C47.2, C48.2, C49.2, C50.2, C51.2, C52.2, C53.2, C54.2, C55.2, C56.2, C57.2, C58.2, C59.2, C6.2, C60.2, C61.2, C62.2, C63.2, C64.2, C65.2, C66.2, C67.2, C68.2, C69.2, C7.2, C8.2, C9.2
- net VCC: now also C10.2, C11.2, C12.2, C13.2, C14.2, C15.2, C16.2, C17.2, C18.2, C19.2, C20.2, C21.2, C22.2, C23.2, C24.2, C25.2, C26.2, C27.2, C28.2, C29.2, C30.2, C31.2, C32.2, C33.2, C34.2, C35.2, C36.2, C37.2, C38.2, C39.2, C40.2, C41.2, C42.2, C43.2, C44.2, C45.2, C46.2, C47.2, C48.2, C49.2, C50.2, C51.2, C52.2, C53.2, C54.2, C55.2, C56.2, C57.2, C58.2, C59.2, C6.2, C60.2, C61.2, C62.2, C63.2, C64.2, C65.2, C66.2, C67.2, C68.2, C69.2, C7.2, C8.2, C9.2, U10.2 (VDD), U11.2 (VDD), U12.2 (VDD), U13.2 (VDD), U14.2 (VDD), U15.2 (VDD), U16.2 (VDD), U17.2 (VDD), U18.2 (VDD), U19.2 (VDD), U20.2 (VDD), U21.2 (VDD), U22.2 (VDD), U23.2 (VDD), U24.2 (VDD), U25.2 (VDD), U26.2 (VDD), U27.2 (VDD), U28.2 (VDD), U29.2 (VDD), U30.2 (VDD), U31.2 (VDD), U32.2 (VDD), U33.2 (VDD), U34.2 (VDD), U35.2 (VDD), U36.2 (VDD), U37.2 (VDD), U38.2 (VDD), U39.2 (VDD), U40.2 (VDD), U41.2 (VDD), U42.2 (VDD), U43.2 (VDD), U44.2 (VDD), U45.2 (VDD), U46.2 (VDD), U47.2 (VDD), U48.2 (VDD), U49.2 (VDD), U50.2 (VDD), U51.2 (VDD), U52.2 (VDD), U53.2 (VDD), U54.2 (VDD), U55.2 (VDD), U56.2 (VDD), U57.2 (VDD), U58.2 (VDD), U59.2 (VDD), U6.2 (VDD), U60.2 (VDD), U61.2 (VDD), U62.2 (VDD), U63.2 (VDD), U64.2 (VDD), U65.2 (VDD), U66.2 (VDD), U67.2 (VDD), U68.2 (VDD), U69.2 (VDD), U7.2 (VDD), U8.2 (VDD), U9.2 (VDD); no longer C10.1, C11.1, C12.1, C13.1, C14.1, C15.1, C16.1, C17.1, C18.1, C19.1, C20.1, C21.1, C22.1, C23.1, C24.1, C25.1, C26.1, C27.1, C28.1, C29.1, C30.1, C31.1, C32.1, C33.1, C34.1, C35.1, C36.1, C37.1, C38.1, C39.1, C40.1, C41.1, C42.1, C43.1, C44.1, C45.1, C46.1, C47.1, C48.1, C49.1, C50.1, C51.1, C52.1, C53.1, C54.1, C55.1, C56.1, C57.1, C58.1, C59.1, C6.1, C60.1, C61.1, C62.1, C63.1, C64.1, C65.1, C66.1, C67.1, C68.1, C69.1, C7.1, C8.1, C9.1
- net at R4.1: now also U11.6 (BIN), U6.4 (DIN)
- new net: U11.4 (DIN), U16.6 (BIN), U6.3 (DO)
- new net: U11.3 (DO), U16.4 (DIN), U21.6 (BIN)
- new net: U16.3 (DO), U21.4 (DIN), U26.6 (BIN)
- new net: U21.3 (DO), U26.4 (DIN), U31.6 (BIN)
- new net: U26.3 (DO), U31.4 (DIN)
- new net: U31.3 (DO), U36.4 (DIN), U41.6 (BIN)
- new net: U36.3 (DO), U41.4 (DIN), U46.6 (BIN)
- new net: U41.3 (DO), U46.4 (DIN), U51.6 (BIN)
- new net: U46.3 (DO), U51.4 (DIN), U56.6 (BIN)
- new net: U51.3 (DO), U56.4 (DIN), U61.6 (BIN)
- new net: U56.3 (DO), U61.4 (DIN), U66.6 (BIN)
- new net: U61.3 (DO), U66.4 (DIN), U7.6 (BIN)
- new net: U12.6 (BIN), U66.3 (DO), U7.4 (DIN)
- new net: U12.4 (DIN), U17.6 (BIN), U7.3 (DO)
- new net: U17.3 (DO), U22.4 (DIN), U27.6 (BIN)
- new net: U12.3 (DO), U17.4 (DIN), U22.6 (BIN)
- new net: U22.3 (DO), U27.4 (DIN), U32.6 (BIN)
- new net: U27.3 (DO), U32.4 (DIN)
- new net: U32.3 (DO), U37.4 (DIN), U42.6 (BIN)
- new net: U37.3 (DO), U42.4 (DIN), U47.6 (BIN)
- new net: U42.3 (DO), U47.4 (DIN), U52.6 (BIN)
- new net: U47.3 (DO), U52.4 (DIN), U57.6 (BIN)
- new net: U52.3 (DO), U57.4 (DIN), U62.6 (BIN)
- new net: U57.3 (DO), U62.4 (DIN), U67.6 (BIN)
- new net: U62.3 (DO), U67.4 (DIN), U8.6 (BIN)
- new net: U13.6 (BIN), U67.3 (DO), U8.4 (DIN)
- new net: U13.4 (DIN), U18.6 (BIN), U8.3 (DO)
- new net: U18.3 (DO), U23.4 (DIN), U28.6 (BIN)
- new net: U13.3 (DO), U18.4 (DIN), U23.6 (BIN)
- new net: U23.3 (DO), U28.4 (DIN), U33.6 (BIN)
- new net: U28.3 (DO), U33.4 (DIN)
- new net: U33.3 (DO), U38.4 (DIN), U43.6 (BIN)
- new net: U38.3 (DO), U43.4 (DIN), U48.6 (BIN)
- new net: U43.3 (DO), U48.4 (DIN), U53.6 (BIN)
- new net: U48.3 (DO), U53.4 (DIN), U58.6 (BIN)
- new net: U53.3 (DO), U58.4 (DIN), U63.6 (BIN)
- new net: U58.3 (DO), U63.4 (DIN), U68.6 (BIN)
- new net: U63.3 (DO), U68.4 (DIN), U9.6 (BIN)
- new net: U14.6 (BIN), U68.3 (DO), U9.4 (DIN)
- new net: U14.4 (DIN), U19.6 (BIN), U9.3 (DO)
- new net: U19.3 (DO), U24.4 (DIN), U29.6 (BIN)
- new net: U14.3 (DO), U19.4 (DIN), U24.6 (BIN)
- new net: U24.3 (DO), U29.4 (DIN), U34.6 (BIN)
- new net: U29.3 (DO), U34.4 (DIN)
- new net: U34.3 (DO), U39.4 (DIN), U44.6 (BIN)
- new net: U39.3 (DO), U44.4 (DIN), U49.6 (BIN)
- new net: U44.3 (DO), U49.4 (DIN), U54.6 (BIN)
- new net: U49.3 (DO), U54.4 (DIN), U59.6 (BIN)
- new net: U54.3 (DO), U59.4 (DIN), U64.6 (BIN)
- new net: U59.3 (DO), U64.4 (DIN), U69.6 (BIN)
- new net: U10.6 (BIN), U64.3 (DO), U69.4 (DIN)
- new net: U10.4 (DIN), U15.6 (BIN), U69.3 (DO)
- new net: U10.3 (DO), U15.4 (DIN), U20.6 (BIN)
- new net: U20.3 (DO), U25.4 (DIN), U30.6 (BIN)
- new net: U15.3 (DO), U20.4 (DIN), U25.6 (BIN)
- new net: U25.3 (DO), U30.4 (DIN), U35.6 (BIN)
- new net: U30.3 (DO), U35.4 (DIN)
- new net: U35.3 (DO), U40.4 (DIN), U45.6 (BIN)
- new net: U40.3 (DO), U45.4 (DIN), U50.6 (BIN)
- new net: U45.3 (DO), U50.4 (DIN), U55.6 (BIN)
- new net: U50.3 (DO), U55.4 (DIN), U60.6 (BIN)
- new net: U55.3 (DO), U60.4 (DIN), U65.6 (BIN)
- new net: U60.3 (DO), U65.4 (DIN)
- no-connect marks 16 -> 80
Other:
- moved on the sheet: C1, C2, C3, C4, C5, C6, C70, D1, FB2, J1, P1, P2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

Commit message: updated pcb layout for ws2813b led
Connections:
- net at U26.3 (DO), U31.4 (DIN): now also U36.6 (BIN)
- net at U27.3 (DO), U32.4 (DIN): now also U37.6 (BIN)
- net at U28.3 (DO), U33.4 (DIN): now also U38.6 (BIN)
- net at U29.3 (DO), U34.4 (DIN): now also U39.6 (BIN)
- net at U30.3 (DO), U35.4 (DIN): now also U40.6 (BIN)
Changed lines of the file:
@@
 Connection ~ 14450 7000
 NoConn ~ 14250 8100
+Wire Wire Line
+	7450 5750 7450 5900
+Connection ~ 7450 5900
+Wire Wire Line
+	7450 4650 7450 4800
+Connection ~ 7450 4800
+Wire Wire Line
+	7450 6850 7450 7000
+Connection ~ 7450 7000
+Wire Wire Line
+	7450 7950 7450 8100
+Connection ~ 7450 8100
+Wire Wire Line
+	7450 3550 7450 3700
+Connection ~ 7450 3700
 $EndSCHEMATC
